File: placa/placa.kicad_sch (KiCad schematic)
At the start: 22 parts, among them J1 Conn_01x02_Socket, J2 Conn_02x02_Top_Bottom, J3 Conn_01x09_Female, J4 Conn_01x02_Female, J5 Conn_01x02_Female, U1 DRV8872DDA, U2 DRV8872DDA, U3 V7805-500

Commit message: *
Parts:
- removed D2: 1N4001, Diode_THT:D_DO-41_SOD81_P10.16mm_Horizontal, symbol Diode:1N4001
- removed J1: Conn_01x02_Socket, symbol Connector:Conn_01x02_Socket
- removed R1, R2, R3, R4: 10k, symbol Device:R
- removed U1, U2: DRV8872DDA, Package_SO:Texas_HTSOP-8-1EP_3.9x4.9mm_P1.27mm_EP2.95x4.9mm_Mask2.4x3.1mm_ThermalVias, symbol Driver_Motor:DRV8872DDA
- removed U3: V7805-500, digikey-footprints:3-SIP_Module_V7805-500, symbol dk_DC-DC-Converters:V7805-500
- added J6, J7: Conn_01x02_Socket, Connector_PinHeader_2.00mm:PinHeader_1x02_P2.00mm_Vertical, symbol Connector:Conn_01x02_Socket
- added J8: Conn_01x02_Socket, Connector_Wire:SolderWire-0.1sqmm_1x02_P3.6mm_D0.4mm_OD1mm_Relief, symbol Connector:Conn_01x02_Socket
- added U1, U2: L7806, Package_TO_SOT_THT:TO-220-3_Vertical, symbol Regulator_Linear:L7806
- C1, C3, C4, C5, C6: footprint (none) -> Capacitor_THT:CP_Radial_D5.0mm_P2.00mm
- C2: value 0.1u -> C; footprint (none) -> Capacitor_THT:CP_Radial_D5.0mm_P2.00mm
- D1: footprint (none) -> LED_THT:LED_D1.8mm_W3.3mm_H2.4mm
- J2: footprint (none) -> Button_Switch_THT:SW_PUSH_6mm
- J3: footprint (none) -> Connector_PinHeader_2.00mm:PinHeader_1x09_P2.00mm_Vertical
- J4, J5: footprint (none) -> Connector_PinHeader_2.00mm:PinHeader_1x02_P2.00mm_Vertical
- R5: footprint (none) -> Resistor_THT:R_Axial_DIN0204_L3.6mm_D1.6mm_P1.90mm_Vertical
Connections:
- net 0: now also C3.2, C4.2, J4.1 (Pin_1), J5.1 (Pin_1), J8.2 (Pin_2), U1.2 (GND), U2.2 (GND)
- net VCC: now also J8.1 (Pin_1); no longer C2.1
- net at A1.19 (A0): now also J6.1 (Pin_1)
- net at A1.20 (A1): now also J6.2 (Pin_2)
- net at A1.21 (A2): now also J7.1 (Pin_1)
- net at A1.22 (A3): now also J7.2 (Pin_2)
- net at A1.27 (+5V), J3.2 (Pin_2): now also C1.1, C2.1, U1.1 (IN), U2.1 (IN)
- net at C4.1, J5.2 (Pin_2): now also U1.3 (OUT)
- net at C3.1, J4.2 (Pin_2): now also U2.3 (OUT)
Other:
- moved on the sheet: C1, C3, J4
