File: modulo sensores.kicad_pcb (KiCad board)
At the start: 2 copper layers, 97.5 x 38.8 mm, 28 parts, among them J1 Conn_01x08_Male, U1 TCMT4106, U2 TCMT4106, U3 TCMT4106, U4 TCMT4106, U5 TCMT4106

Commit message: *
Parts:
- moved 10u1 1.65 mm to (163.1, 100.8), turned to 0 degrees
Routing:
- net Net-(74hc14d1-Pad9): track 120.5 -> 12.4 mm
- net Net-(74hc14d1-Pad10): track 73.6 -> 8.45 mm
- net Net-(74hc14d1-Pad4): track 46.5 -> 10.2 mm
- net VCC: track 209.1 -> 177.7 mm
- net Net-(74hc14d1-Pad1): track 30.2 -> 26.4 mm
- net Net-(74hc14d1-Pad6): track 59.0 -> 56.1 mm
- net Net-(74hc14d1-Pad2): track 51.8 -> 53.2 mm
- net Net-(74hc14d1-Pad8): track 77.4 -> 78.6 mm
- removed copper zone on B.Cu, net GND
